File: ELECTRONICA/MAXPOWER/MAXPOWER.sch (KiCad schematic (older format))
At the start: 10 parts, among them J1 Conn_01x05, J2 Conn_01x05, U1 ATmega2560-16AU

Commit message: kicad pines de expansion
Parts:
- added D2: LED, symbol Device:LED
- added J10: Conn_01x04_MMA8451, symbol Connector_Generic:Conn_01x04
- added J11: Conn_01x08_LSM303, symbol Connector_Generic:Conn_01x08
- added J12: Conn_01x04_OLED, symbol Connector_Generic:Conn_01x04
- added J13: Conn_01x04_EXTRA, symbol Connector_Generic:Conn_01x04
- added J14, J15, J16, J17: Conn_01x03_TMP, symbol Connector_Generic:Conn_01x03
- added J18: Conn_01x03_LDR, symbol Connector_Generic:Conn_01x03
- added J19: Conn_01x03_FAST_LED, symbol Connector_Generic:Conn_01x03
- added J20: Conn_01x04_LED_EXTRA, symbol Connector_Generic:Conn_01x04
- added J21: Conn_01x06_M1, symbol Connector_Generic:Conn_01x07
- added J22: Conn_01x06_M2, symbol Connector_Generic:Conn_01x07
- added J23: Conn_01x05_M3, symbol Connector_Generic:Conn_01x07
- added J24: Conn_01x05_M4, symbol Connector_Generic:Conn_01x07
- added J25: ENCODERS, symbol Connector_Generic:Conn_01x04
- added J26, J27, J28: Conn_01x21_exp, symbol Connector_Generic:Conn_01x21
- added J3: Conn_01x06_SPI, symbol Connector_Generic:Conn_01x06
- added J4: Conn_02x03_ICSP, symbol Connector_Generic:Conn_02x03_Top_Bottom
- added J5: Conn_02x04_WIFI_ESP, symbol Connector_Generic:Conn_02x04_Top_Bottom
- added J6: Conn_01x04_SERIAL2, symbol Connector_Generic:Conn_01x04
- added J7: Conn_01x04_SERIAL1, symbol Connector_Generic:Conn_01x04
- added J8: Conn_01x04_SI7021, symbol Connector_Generic:Conn_01x04
- added J9: Conn_01x04_BMP180, symbol Connector_Generic:Conn_01x04
- added Q1, Q2, Q3: IRF540N, Package_TO_SOT_THT:TO-220-3_Vertical, symbol Transistor_FET:IRF540N
- added R10, R12, R14, R4, R5, R9: 10K, symbol Device:R
- added R11, R13, R15, R7: 1K, symbol Device:R
- added R16: 330, symbol Device:R
- added R6: 2K, symbol Device:R
- added R8: 10k, symbol Device:R
- added RV1: R_POT, symbol Device:R_POT
- added SW1: SW_DPDT_x2_TX0, symbol Switch:SW_DPDT_x2
- added SW10: SW_DIP_x08, symbol Switch:SW_DIP_x08
- added SW2: SW_DPDT_x2_RX0, symbol Switch:SW_DPDT_x2
- added SW3: SW_SP3T_RESET, symbol Switch:SW_SP3T
- added SW4: SW_DPDT_x2_WIFI_LOAD_EXE, symbol Switch:SW_DPDT_x2
- added SW5: UP, symbol Switch:SW_Push
- added SW6: RIGHT, symbol Switch:SW_Push
- added SW7: LEFT, symbol Switch:SW_Push
- added SW8: OK, symbol Switch:SW_Push
- added SW9: DOWN, symbol Switch:SW_Push
- added U2: 74LS247, symbol 74xx:74LS247
- added U3: CC56-12SYKWA, Display_7Segment:CA56-12SYKWA, symbol Display_Character:CC56-12SYKWA
- J1: value Conn_01x05 -> Conn_01x05_Bluetooth
- J2: value Conn_01x05 -> Conn_01x05_FTDI
Connections:
- net +5V: now also J10.1 (Pin_1), J11.7 (Pin_7), J12.3 (Pin_3), J13.3 (Pin_3), J14.1 (Pin_1), J15.1 (Pin_1), J16.1 (Pin_1), J17.1 (Pin_1), J18.1 (Pin_1), J19.1 (Pin_1), J21.1 (Pin_1), J22.1 (Pin_1), J23.1 (Pin_1), J24.1 (Pin_1), J27.1 (Pin_1), J27.10 (Pin_10), J27.11 (Pin_11), J27.12 (Pin_12), J27.13 (Pin_13), J27.14 (Pin_14), J27.15 (Pin_15), J27.16 (Pin_16), J27.17 (Pin_17), J27.18 (Pin_18), J27.19 (Pin_19), J27.2 (Pin_2), J27.20 (Pin_20), J27.21 (Pin_21), J27.3 (Pin_3), J27.4 (Pin_4), J27.5 (Pin_5), J27.6 (Pin_6), J27.7 (Pin_7), J27.8 (Pin_8), J27.9 (Pin_9), J3.2 (Pin_2), J4.4 (Pin_4), J5.3 (Pin_3), J5.4 (Pin_4), J6.2 (Pin_2), J7.2 (Pin_2), J8.3 (Pin_3), J9.4 (Pin_4), R4.1, R5.1, R8.1, R9.1, RV1.1, SW4.1 (A), U2.16 (VCC), U2.3 (Lt), U2.5 (Rbi)
- net Earth: now also R2.2, D2.1 (K), J10.4 (Pin_4), J11.8 (Pin_8), J12.4 (Pin_4), J13.4 (Pin_4), J14.3 (Pin_3), J15.3 (Pin_3), J16.3 (Pin_3), J17.3 (Pin_3), J18.3 (Pin_3), J19.3 (Pin_3), J20.4 (Pin_4), J21.2 (Pin_2), J21.3 (Pin_3), J22.2 (Pin_2), J22.3 (Pin_3), J23.2 (Pin_2), J23.3 (Pin_3), J24.2 (Pin_2), J24.3 (Pin_3), J28.1 (Pin_1), J28.10 (Pin_10), J28.11 (Pin_11), J28.12 (Pin_12), J28.13 (Pin_13), J28.14 (Pin_14), J28.15 (Pin_15), J28.16 (Pin_16), J28.17 (Pin_17), J28.18 (Pin_18), J28.19 (Pin_19), J28.2 (Pin_2), J28.20 (Pin_20), J28.21 (Pin_21), J28.3 (Pin_3), J28.4 (Pin_4), J28.5 (Pin_5), J28.6 (Pin_6), J28.7 (Pin_7), J28.8 (Pin_8), J28.9 (Pin_9), J3.1 (Pin_1), J4.6 (Pin_6), J5.5 (Pin_5), J6.1 (Pin_1), J7.1 (Pin_1), J8.4 (Pin_4), J9.3 (Pin_3), Q1.3 (S), Q2.3 (S), Q3.3 (S), R10.2, R12.2, R14.2, R6.1, RV1.3, SW10.1, SW10.2, SW10.3, SW10.4, SW10.5, SW10.6, SW10.7, SW10.8, SW4.3 (C), SW5.1, SW6.1, SW7.1, SW8.1, SW9.1, U2.8 (GND); no longer R2.1
- net RX0: now also U1.2 (PE0), SW2.2 (B)
- net TX0: now also U1.3 (PE1), SW1.2 (B)
- net R_LED: now reaches U1.1 (PG5)
- net R_LED: now also R15.1
- net RX2: now reaches U1.12 (PH0)
- net RX2: now also J7.4 (Pin_4), R7.1
- net TX2: now reaches U1.13 (PH1)
- net TX2: now also J5.8 (Pin_8), J7.3 (Pin_3)
- net PH2: now reaches U1.14 (PH2)
- net PH2: now also J26.8 (Pin_8)
- net PWM4: now reaches U1.15 (PH3)
- net PWM4: now also J24.7 (Pin_7)
- net PWMH1: now reaches U1.16 (PH4)
- net PWMH1: now also J26.1 (Pin_1)
- net PWMH2: now reaches U1.17 (PH5)
- net PWMH2: now also J26.2 (Pin_2)
- net PH6: now reaches U1.18 (PH6)
- net PH6: now also J26.9 (Pin_9)
- net SS: now reaches U1.19 (PB0)
- net SS: now also J3.3 (Pin_3)
- net SCK: now reaches U1.20 (PB1)
- net SCK: now also J3.6 (Pin_6), J4.2 (Pin_2)
- net MOSI: now reaches U1.21 (PB2)
- net MOSI: now also J3.4 (Pin_4), J4.5 (Pin_5)
- net MISO: now reaches U1.22 (PB3)
- net MISO: now also J3.5 (Pin_5), J4.1 (Pin_1)
- net G_LED: now reaches U1.23 (PB4)
- net G_LED: now also R13.1
- net B_LED: now reaches U1.24 (PB5)
- net B_LED: now also R11.1
- net FAST_LED: now reaches U1.25 (PB6)
- net FAST_LED: now also J19.2 (Pin_2)
- net at U1.26 (PB7): now also R16.2
- net PH7: now reaches U1.27 (PH7)
- net PH7: now also J26.10 (Pin_10)
- net PG3: now reaches U1.28 (PG3)
- net PG3: now also J26.14 (Pin_14)
- net PG4: now reaches U1.29 (PG4)
- net PG4: now also J26.15 (Pin_15)
- net UP: now reaches U1.35 (PL0)
- net UP: now also SW5.2
- net RIGHT: now reaches U1.36 (PL1)
- net RIGHT: now also SW6.2
- net LEFT: now reaches U1.37 (PL2)
- net LEFT: now also SW7.2
- net OK: now reaches U1.38 (PL3)
- net OK: now also SW8.2
- net DOWN: now reaches U1.39 (PL4)
- net DOWN: now also SW9.2
- net PWML1: now reaches U1.40 (PL5)
- net PWML1: now also J26.3 (Pin_3)
- net PWML2: now reaches U1.41 (PL6)
- net PWML2: now also J26.4 (Pin_4)
- net PWML3: now reaches U1.42 (PL7)
- net PWML3: now also J26.5 (Pin_5)
- net SCL: now reaches U1.43 (PD0)
- net SCL: now also J10.2 (Pin_2), J11.3 (Pin_3), J12.2 (Pin_2), J13.2 (Pin_2), J8.1 (Pin_1), J9.2 (Pin_2), R8.2
- net SDA: now reaches U1.44 (PD1)
- net SDA: now also J10.3 (Pin_3), J11.2 (Pin_2), J12.1 (Pin_1), J13.1 (Pin_1), J8.2 (Pin_2), J9.1 (Pin_1), R9.2
- net RX1: now reaches U1.45 (PD2)
- net RX1: now also J6.4 (Pin_4)
- net TX1: now reaches U1.46 (PD3)
- net TX1: now also J6.3 (Pin_3)
- net PD4: now reaches U1.47 (PD4)
- net PD4: now also J26.16 (Pin_16)
- net PD5: now reaches U1.48 (PD5)
- net PD5: now also J26.17 (Pin_17)
- net PD6: now reaches U1.49 (PD6)
- net PD6: now also J26.18 (Pin_18)
- net PWM1: now reaches U1.5 (PE3)
- net PWM1: now also J21.7 (Pin_7)
- net PD7: now reaches U1.50 (PD7)
- net PD7: now also J26.19 (Pin_19)
- net PG0: now reaches U1.51 (PG0)
- net PG0: now also J26.11 (Pin_11)
- net PG1: now reaches U1.52 (PG1)
- net PG1: now also J26.12 (Pin_12)
- net DISPLAY_A: now reaches U1.53 (PC0)
- net DISPLAY_A: now also U2.7 (A)
- net DISPLAY_B: now reaches U1.54 (PC1)
- net DISPLAY_B: now also U2.1 (B)
- net DISPLAY_C: now reaches U1.55 (PC2)
- net DISPLAY_C: now also U2.2 (C)
- net DISPLAY_D: now reaches U1.56 (PC3)
- net DISPLAY_D: now also U2.6 (D)
- net DISPLAY_1: now reaches U1.57 (PC4)
- net DISPLAY_1: now also U3.12 (CC1)
- net DISPLAY_2: now reaches U1.58 (PC5)
- net DISPLAY_2: now also U3.9 (CC2)
- net DISPLAY_3: now reaches U1.59 (PC6)
- net DISPLAY_3: now also U3.8 (CC3)
- net PWM2: now reaches U1.6 (PE4)
- net PWM2: now also J22.7 (Pin_7)
- net DISPLAY_4: now reaches U1.60 (PC7)
- net DISPLAY_4: now also U3.6 (CC4)
- net at U1.63 (PJ0): now also SW10.16
- net at U1.64 (PJ1): now also SW10.15
- net at U1.65 (PJ2): now also SW10.14
- net at U1.66 (PJ3): now also SW10.13
- net at U1.67 (PJ4): now also SW10.12
- net at U1.68 (PJ5): now also SW10.11
- net at U1.69 (PJ6): now also SW10.10
- net PWM3: now reaches U1.7 (PE5)
- net PWM3: now also J23.7 (Pin_7)
- net PG2: now reaches U1.70 (PG2)
- net PG2: now also J26.13 (Pin_13)
- net INB4: now reaches U1.71 (PA7)
- net INB4: now also J24.6 (Pin_6)
- net INB3: now reaches U1.72 (PA6)
- net INB3: now also J23.6 (Pin_6)
- net INB2: now reaches U1.73 (PA5)
- net INB2: now also J22.6 (Pin_6)
- net INB1: now reaches U1.74 (PA4)
- net INB1: now also J21.6 (Pin_6)
- net INA4: now reaches U1.75 (PA3)
- net INA4: now also J24.5 (Pin_5)
- net INA3: now reaches U1.76 (PA2)
- net INA3: now also J23.5 (Pin_5)
- net INA2: now reaches U1.77 (PA1)
- net INA2: now also J22.5 (Pin_5)
- net INA1: now reaches U1.78 (PA0)
- net INA1: now also J21.5 (Pin_5)
- net at U1.79 (PJ7): now also SW10.9
- net PE6: now reaches U1.8 (PE6)
- net PE6: now also J26.20 (Pin_20)
- net PK7: now reaches U1.82 (PK7)
- net PK7: now also J26.7 (Pin_7)
- net PK6: now reaches U1.83 (PK6)
- net PK6: now also J26.6 (Pin_6)
- net LDR: now reaches U1.84 (PK5)
- net LDR: now also J18.2 (Pin_2)
- net TMP4: now reaches U1.85 (PK4)
- net TMP4: now also J17.2 (Pin_2)
- net TMP3: now reaches U1.86 (PK3)
- net TMP3: now also J16.2 (Pin_2)
- net TMP2: now reaches U1.87 (PK2)
- net TMP2: now also J15.2 (Pin_2)
- net TMP1: now reaches U1.88 (PK1)
- net TMP1: now also J14.2 (Pin_2)
- net POT: now reaches U1.89 (PK0)
- net POT: now also RV1.2
- net PE7: now reaches U1.9 (PE7)
- net PE7: now also J26.21 (Pin_21)
- net at U1.90 (PF7): now also J25.4 (Pin_4)
- net at U1.91 (PF6): now also J25.3 (Pin_3)
- net at U1.92 (PF5): now also J25.2 (Pin_2)
- net at U1.93 (PF4): now also J25.1 (Pin_1)
- net CS4: now reaches U1.94 (PF3)
- net CS4: now also J24.4 (Pin_4)
- net CS3: now reaches U1.95 (PF2)
- net CS3: now also J23.4 (Pin_4)
- net CS2: now reaches U1.96 (PF1)
- net CS2: now also J22.4 (Pin_4)
- net CS1: now reaches U1.97 (PF0)
- net CS1: now also J21.4 (Pin_4)
- net RESET_Bluetooth: now reaches J1.1 (Pin_1)
- net RESET_Bluetooth: now also J2.1 (Pin_1), R2.1, R3.2, SW3.2, SW3.4
- net TX: now reaches J1.2 (Pin_2)
- net TX: now also J2.2 (Pin_2), SW2.1 (A), SW2.3 (C)
- net RX: now reaches J1.3 (Pin_3)
- net RX: now also J2.3 (Pin_3), SW1.1 (A), SW1.3 (C)
- removed net RESET: J2.3 (Pin_3), R2.2, R3.2, U1.30 (~RESET)
- new net: SW3.3, U1.30 (~RESET)
- new net: J5.1 (Pin_1), R6.2, R7.2
- new net: J5.2 (Pin_2), SW4.2 (B)
- new net: J5.6 (Pin_6), R4.2
- new net: J5.7 (Pin_7), R5.2
- new net: D2.2 (A), R16.1
- new net: J20.1 (Pin_1), Q3.2 (D)
- new net: J20.2 (Pin_2), Q2.2 (D), Q3.1 (G), R14.1, R15.2
- new net: J20.3 (Pin_3), Q1.2 (D)
- new net: Q2.1 (G), R12.1, R13.2
- new net: Q1.1 (G), R10.1, R11.2
- new net: U2.9 (e), U3.1 (e)
- new net: U2.15 (f), U3.10 (f)
- new net: U2.13 (a), U3.11 (a)
- new net: U2.10 (d), U3.2 (d)
- new net: U2.4 (Rbo), U3.3 (DPX)
- new net: U2.11 (c), U3.4 (c)
- new net: U2.14 (g), U3.5 (g)
- new net: U2.12 (b), U3.7 (b)
- new net RESET_ICSP: J4.3 (Pin_3), SW3.1
Other:
- moved on the sheet: 16MHz1, C1, C2, D1, J1, J2, R1, R2, R3, U1

Commit message: kicad motor encoders
Parts:
- added C10, C7, C8, C9: 1mF, symbol Device:C
- added C3, C4, C5, C6: 27nF, symbol Device:C
- added R17, R18, R19, R20: 24K, symbol Device:R
- added R21, R22, R23, R24: 1K, symbol Device:R
- added U10, U11, U8, U9: LM2907, LM2907:SOIC8, symbol LM2907:LM2907
- added U4, U5, U6, U7: HEF4040BT, HEF4040BT:SOIC127P600X175-16N, symbol HEF4040BT:HEF4040BT
- J26, J27, J28: value Conn_01x21_exp -> Conn_01x22_exp; symbol Connector_Generic:Conn_01x21 -> Connector_Generic:Conn_01x22
Connections:
- net +5V: now also J27.22 (Pin_22), U10.5, U10.6 (6_VCC), U11.5, U11.6 (6_VCC), U4.16 (VDD), U5.16 (VDD), U6.16 (VDD), U7.16 (VDD), U8.5, U8.6 (6_VCC), U9.5, U9.6 (6_VCC)
- net Earth: now also J28.22 (Pin_22), C10.1, C3.1, C4.1, C5.1, C6.1, C7.1, C8.1, C9.1, R17.2, R18.2, R19.2, R20.2, R21.1, R22.1, R23.1, R24.1, U10.8, U11.8, U4.11 (MR), U4.8 (VSS), U5.11 (MR), U5.8 (VSS), U6.11 (MR), U6.8 (VSS), U7.11 (MR), U7.8 (VSS), U8.8, U9.8
- net PE6: now also J26.21 (Pin_21); no longer J26.20 (Pin_20)
- net PE7: now also J26.22 (Pin_22); no longer J26.21 (Pin_21)
- net PE2: now reaches U1.4 (PE2)
- net PE2: now also J26.20 (Pin_20)
- net EN4: now reaches U1.90 (PF7)
- net EN4: now also R22.2, U9.4, U9.7; no longer J25.4 (Pin_4)
- net EN3: now reaches U1.91 (PF6)
- net EN3: now also R21.2, U8.4, U8.7; no longer J25.3 (Pin_3)
- net EN2: now reaches U1.92 (PF5)
- net EN2: now also R24.2, U11.4, U11.7; no longer J25.2 (Pin_2)
- net EN1: now reaches U1.93 (PF4)
- net EN1: now also R23.2, U10.4, U10.7; no longer J25.1 (Pin_1)
- new net: C4.2, U9.2
- new net: C8.2, R18.1, U9.3
- new net: C3.2, U8.2
- new net: C7.2, R17.1, U8.3
- new net: C5.2, U10.2
- new net: C9.2, R19.1, U10.3
- new net: C6.2, U11.2
- new net: C10.2, R20.1, U11.3
- new net EN_IN1: J25.4 (Pin_4), U4.10 (~CP)
- new net EN_IN2: J25.3 (Pin_3), U5.10 (~CP)
- new net EN_IN3: J25.2 (Pin_2)
- new net EN_IN4: J25.1 (Pin_1), U6.10 (~CP), U7.10 (~CP)
- new net EN_T1: U10.1 (1_VIN), U4.2 (Q5)
- new net EN_T2: U11.1 (1_VIN), U5.2 (Q5)
- new net EN_T3: U6.2 (Q5), U8.1 (1_VIN)
- new net EN_T4: U7.2 (Q5), U9.1 (1_VIN)
Other:
- moved on the sheet: J10, J11, J12, J13, J14, J15, J16, J17, J18, J21, J22, J23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

Commit message: kicad opencv
Parts:
- removed C10, C7, C8, C9: 1mF, symbol Device:C
- removed C3, C5, C6: 27nF, symbol Device:C
- removed J7: Conn_01x04_SERIAL1, symbol Connector_Generic:Conn_01x04
- removed SW1: SW_DPDT_x2_TX0, symbol Switch:SW_DPDT_x2
- removed SW2: SW_DPDT_x2_RX0, symbol Switch:SW_DPDT_x2
- removed SW3: SW_SP3T_RESET, symbol Switch:SW_SP3T
- removed SW4: SW_DPDT_x2_WIFI_LOAD_EXE, symbol Switch:SW_DPDT_x2
- added C10, C29, C30, C9: e1uF, Capacitor_SMD:CP_Elec_4x5.3, symbol Device:CP
- added C11, C13, C14, C15, C16, C17, C18, C19, C20, C21, C22, C23, C24, C25, C26, C27, C28, C32, C34, C36: 100nF, Capacitor_SMD:C_0805_2012Metric_Pad1.15x1.40mm_HandSolder, symbol Device:C
- added C12: 220nF, Capacitor_SMD:C_0805_2012Metric_Pad1.15x1.40mm_HandSolder, symbol Device:C
- added C3, C31, C33, C35: e47uF, Capacitor_SMD:CP_Elec_6.3x5.3, symbol Device:CP
- added C5, C6, C7, C8: e100nF, Capacitor_SMD:CP_Elec_4x5.3, symbol Device:CP
- added D3, D4, D5, D6, D7: D, other:DO-214AA, symbol Device:D
- added J29: HOLE1, huellas:hole, symbol Connector_Generic:Conn_01x01
- added J30: HOLE2, huellas:hole, symbol Connector_Generic:Conn_01x01
- added J31: HOLE3, huellas:hole, symbol Connector_Generic:Conn_01x01
- added J32: HOLE4, huellas:hole, symbol Connector_Generic:Conn_01x01
- added J33: Conn_01x04_LED_EXTRA, symbol Connector_Generic:Conn_01x04
- added J34, J35, J36: ENCODERS, symbol Connector_Generic:Conn_01x04
- added J37: Conn_01x02_INPUT, proyectoAjeno:XT30PW-F2, symbol Connector_Generic:Conn_01x02
- added J38: Conn_01x04, symbol Connector_Generic:Conn_01x04
- added J39: JUMPER_WIFI, symbol Connector_Generic:Conn_01x03
- added J7: Conn_01x05_Bluetooth_COMM, symbol Connector_Generic:Conn_01x05
- added LED1, LED10, LED11, LED12, LED13, LED14, LED15, LED16, LED2, LED3, LED4, LED5, LED6, LED7, LED8, LED9: WS2812B, WS2812B:WS2812B_data-bridgeable, symbol ws2812b:WS2812B
- added R25: 10K, Resistor_SMD:R_0805_2012Metric_Pad1.15x1.40mm_HandSolder, symbol Device:R
- added SW1: RESET, huellas:PULSADOR, symbol Switch:SW_Push
- added U12, U13: L7805, Compluino_03:7805, symbol Regulator_Linear:L7805
- 16MHz1: footprint (none) -> Compluino_03:Crystal
- C1, C2: footprint (none) -> Capacitor_SMD:C_0805_2012Metric_Pad1.15x1.40mm_HandSolder
- C4: value 27nF -> 100nF; footprint (none) -> Capacitor_SMD:C_0805_2012Metric_Pad1.15x1.40mm_HandSolder
- D1, D2: footprint (none) -> LED_SMD:LED_1210_3225Metric_Pad1.42x2.65mm_HandSolder
- J12: footprint (none) -> Compluino_03:OLED
- J20: value Conn_01x04_LED_EXTRA -> Conn_01x04
- Q1, Q2, Q3: footprint Package_TO_SOT_THT:TO-220-3_Vertical -> other:D2PAK
- R1, R16: value 330 -> 249; footprint (none) -> Resistor_SMD:R_0805_2012Metric_Pad1.15x1.40mm_HandSolder
- R10, R11, R12, R13, R14, R15, R2, R21, R22, R23, R24, R3, R4, R5, R6, R7, R8, R9: footprint (none) -> Resistor_SMD:R_0805_2012Metric_Pad1.15x1.40mm_HandSolder
- R17, R18, R19, R20: value 24K -> 11,3K; footprint (none) -> Resistor_SMD:R_0805_2012Metric_Pad1.15x1.40mm_HandSolder
- RV1: footprint (none) -> Compluino_03:Potenciometro
- SW10: footprint (none) -> huellas:SWITCH
- SW5, SW6, SW7, SW8, SW9: footprint (none) -> huellas:PULSADOR
- U2: footprint (none) -> other:SO16
Connections:
- net RESET_ICSP is gone; now on net RESET_Bluetooth: J4.3 (Pin_3)
- net RX is gone; now on net TX0: J1.3 (Pin_3), J2.3 (Pin_3)
- net RX2 is gone; now on net RX0: R7.1, U1.12 (PH0)
- net TX is gone; now on net RX0: J1.2 (Pin_2), J2.2 (Pin_2)
- net TX2 is gone; now on net TX0: J5.8 (Pin_8), U1.13 (PH1)
- net +5V: now also J25.3 (Pin_3), C33.1, C34.2, J34.3 (Pin_3), J35.3 (Pin_3), J36.3 (Pin_3), J39.1 (Pin_1), J7.5 (Pin_5), R25.1, U13.3 (OUT); no longer J19.1 (Pin_1), U1.10 (VCC), U1.100 (AVCC), U1.31 (VCC), U1.61 (VCC), U1.80 (VCC), U10.5, U10.6 (6_VCC), U11.5, U11.6 (6_VCC), U8.5, U8.6 (6_VCC), U9.5, U9.6 (6_VCC)
- net EN_IN1: now also J25.2 (Pin_2); no longer J25.4 (Pin_4)
- net EN_IN2: now also J35.2 (Pin_2); no longer J25.3 (Pin_3)
- net EN_IN3: now also J34.2 (Pin_2); no longer J25.2 (Pin_2)
- net EN_IN4: now also J36.2 (Pin_2); no longer J25.1 (Pin_1)
- net EN_T1: now also U4.4 (Q6); no longer U4.2 (Q5)
- net EN_T2: now also U5.4 (Q6); no longer U5.2 (Q5)
- net EN_T3: now also U6.4 (Q6); no longer U6.2 (Q5)
- net EN_T4: now also U7.4 (Q6); no longer U7.2 (Q5)
- net Earth: now also J20.2 (Pin_2), J20.3 (Pin_3), J25.4 (Pin_4), C10.2, C11.2, C13.2, C14.2, C15.2, C16.2, C17.2, C18.2, C19.2, C20.2, C21.2, C22.2, C23.2, C24.2, C25.2, C26.2, C27.2, C28.2, C29.2, C3.2, C30.2, C31.2, C32.1, C33.2, C34.1, C35.2, C36.1, C5.2, C6.2, C7.2, C8.2, C9.2, J33.1 (Pin_1), J34.4 (Pin_4), J35.4 (Pin_4), J36.4 (Pin_4), J37.2 (Pin_2), J38.2 (Pin_2), J38.3 (Pin_3), J39.3 (Pin_3), J7.4 (Pin_4), LED1.3 (GND), LED10.3 (GND), LED11.3 (GND), LED12.3 (GND), LED13.3 (GND), LED14.3 (GND), LED15.3 (GND), LED16.3 (GND), LED2.3 (GND), LED3.3 (GND), LED4.3 (GND), LED5.3 (GND), LED6.3 (GND), LED7.3 (GND), LED8.3 (GND), LED9.3 (GND), SW1.2, U12.2 (GND), U13.2 (GND); no longer J20.4 (Pin_4), Q1.3 (S), Q2.3 (S), Q3.3 (S), R10.2, R12.2, R14.2
- net FAST_LED: now also LED1.4 (DIN)
- net RESET_Bluetooth: now also C12.2, J7.1 (Pin_1)
- net RX0: now also J7.2 (Pin_2)
- net TX0: now also J7.3 (Pin_3)
- net at U1.30 (~RESET): now also C12.1, C13.1, R25.2, SW1.1
- net at J5.2 (Pin_2): now also J39.2 (Pin_2)
- net at U9.2: now also C6.1; no longer C4.2
- net at R18.1, U9.3: now also C10.1
- net at U8.2: now also C5.1
- net at R17.1, U8.3: now also C9.1
- net at U10.2: now also C7.1
- net at R19.1, U10.3: now also C29.1
- net at U11.2: now also C8.1
- net at R20.1, U11.3: now also C30.1
- net +12V: now reaches Q3.2 (D)
- net +12V: now also Q1.2 (D), Q2.2 (D), U10.5, U10.6 (6_VCC), U11.5, U11.6 (6_VCC), U8.5, U8.6 (6_VCC), U9.5, U9.6 (6_VCC), C35.1, C36.2, J38.1 (Pin_1); no longer J20.1 (Pin_1)
- net at Q3.1 (G), R14.1, R15.2: no longer J20.2 (Pin_2), Q2.2 (D)
- new net: D4.1 (K), D6.1 (K), J38.4 (Pin_4)
- new net: D5.1 (K), U12.1 (IN)
- new net: LED2.2 (DOUT), LED3.4 (DIN)
- new net: LED1.2 (DOUT), LED2.4 (DIN)
- new net: J33.3 (Pin_3), Q2.3 (S), R12.2
- new net: J33.2 (Pin_2), Q3.3 (S), R14.2
- new net: J33.4 (Pin_4), Q1.3 (S), R10.2
- new net: D3.1 (K), J20.4 (Pin_4)
- new net: LED3.2 (DOUT), LED4.4 (DIN)
- new net: LED4.2 (DOUT), LED5.4 (DIN)
- new net: LED5.2 (DOUT), LED6.4 (DIN)
- new net: LED6.2 (DOUT), LED7.4 (DIN)
- new net: LED7.2 (DOUT), LED8.4 (DIN)
- new net: LED10.4 (DIN), LED9.2 (DOUT)
- new net: LED10.2 (DOUT), LED11.4 (DIN)
- new net: LED11.2 (DOUT), LED12.4 (DIN)
- new net: LED12.2 (DOUT), LED13.4 (DIN)
- new net: LED13.2 (DOUT), LED14.4 (DIN)
- new net: LED14.2 (DOUT), LED15.4 (DIN)
- new net: LED15.2 (DOUT), LED16.4 (DIN)
- new net: D7.1 (K), U13.1 (IN)
- new net +5VL: C11.1, C14.1, C15.1, C16.1, C17.1, C18.1, C19.1, C20.1, C21.1, C22.1, C23.1, C24.1, C25.1, C26.1, C27.1, C28.1, C3.1, C4.2, J19.1 (Pin_1), J20.1 (Pin_1), LED1.1 (VCC), LED10.1 (VCC), LED11.1 (VCC), LED12.1 (VCC), LED13.1 (VCC), LED14.1 (VCC), LED15.1 (VCC), LED16.1 (VCC), LED2.1 (VCC), LED3.1 (VCC), LED4.1 (VCC), LED5.1 (VCC), LED6.1 (VCC), LED7.1 (VCC), LED8.1 (VCC), LED9.1 (VCC)
- new net +5VP: C31.1, C32.2, U1.10 (VCC), U1.100 (AVCC), U1.31 (VCC), U1.61 (VCC), U1.80 (VCC), U12.3 (OUT)
- new net VCC: D3.2 (A), D4.2 (A), D5.2 (A), D6.2 (A), D7.2 (A), J37.1 (Pin_1)
Other:
- moved on the sheet: J19, J25, J26, J27, J28, Q1, Q2, Q3, R10, R11, R12, R13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
