File: ELECTRONICA/MAXPOWER/MAXPOWER.sch (KiCad schematic (older format))
At the start: 148 parts, among them J1 Conn_01x05_Bluetooth, J10 Conn_01x04_MMA8451, J11 Conn_01x08_LSM303, J12 Conn_01x04_OLED, J13 Conn_01x04_EXTRA, J14 Conn_01x03_TMP, J15 Conn_01x03_TMP, J16 Conn_01x03_TMP, J17 Conn_01x03_TMP, J18 Conn_01x03_LDR, J19 Conn_01x03_FAST_LED, J2 Conn_01x05_FTDI, J20 Conn_01x04, J21 Conn_01x06_M1, J22 Conn_01x06_M2, J23 Conn_01x05_M3, J24 Conn_01x05_M4, J25 ENCODERS, J26 Conn_01x22_exp, J27 Conn_01x22_exp, J28 Conn_01x22_exp, J29 HOLE1, J3 Conn_01x06_SPI, J30 HOLE2, J31 HOLE3, J32 HOLE4, J33 Conn_01x04_LED_EXTRA, J34 ENCODERS, J35 ENCODERS, J36 ENCODERS, J37 Conn_01x02_INPUT, J38 Conn_01x04, J39 JUMPER_WIFI, J4 Conn_02x03_ICSP, J5 Conn_02x04_WIFI_ESP, J6 Conn_01x04_SERIAL2, J7 Conn_01x05_Bluetooth_COMM, J8 Conn_01x04_SI7021, J9 Conn_01x04_BMP180, Q1 IRF540N, Q2 IRF540N, Q3 IRF540N, SW1 RESET, SW10 SW_DIP_x08, SW5 UP, SW6 RIGHT, SW7 LEFT, SW8 OK, SW9 DOWN, U1 ATmega2560-16AU, U10 LM2907, U11 LM2907, U12 L7805, U13 L7805, U2 74LS247, U3 CC56-12SYKWA, U4 HEF4040BT, U5 HEF4040BT, U6 HEF4040BT, U7 HEF4040BT, U8 LM2907, U9 LM2907

Commit message: placa ATtiny1634
Parts:
- removed C10, C29, C30, C9: e1uF, Capacitor_SMD:CP_Elec_4x5.3, symbol Device:CP
- removed C5, C6, C7, C8: e100nF, Capacitor_SMD:CP_Elec_4x5.3, symbol Device:CP
- removed J1: Conn_01x05_Bluetooth, symbol Connector_Generic:Conn_01x05
- removed R17, R18, R19, R20: 11,3K, Resistor_SMD:R_0805_2012Metric_Pad1.15x1.40mm_HandSolder, symbol Device:R
- removed R2, R3: 10K, Resistor_SMD:R_0805_2012Metric_Pad1.15x1.40mm_HandSolder, symbol Device:R
- removed R21, R22, R23, R24: 1K, Resistor_SMD:R_0805_2012Metric_Pad1.15x1.40mm_HandSolder, symbol Device:R
- removed U10, U11, U8, U9: LM2907, LM2907:SOIC8, symbol LM2907:LM2907
- removed U4, U5, U6, U7: HEF4040BT, HEF4040BT:SOIC127P600X175-16N, symbol HEF4040BT:HEF4040BT
- J7: value Conn_01x05_Bluetooth_COMM -> Conn_01x06_Bluetooth_COMM; symbol Connector_Generic:Conn_01x05 -> Connector_Generic:Conn_01x06
Connections:
- net EN_B1: now reaches J25.1 (Pin_1)
- net EN_B2: now reaches J35.1 (Pin_1)
- net EN_B3: now reaches J34.1 (Pin_1)
- net EN_B4: now reaches J36.1 (Pin_1)
- net EN_IN1 renamed EN_A1
- net EN_IN2 renamed EN_A2
- net EN_IN3 renamed EN_A3
- net EN_IN4 renamed EN_A4
- net RESET_Bluetooth renamed RESET_FTDI
- new net ENABLE: J7.6 (Pin_6)
Other:
- moved on the sheet: 16MHz1, C1, C11, C12, C13, C14, C15, C16, C17, C18, C19, C2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
