File: ELECTRONICA/MAXPOWER/MAXPOWER.kicad_pcb (KiCad board)
At the start: 2 copper layers, 2 parts

Commit message: solid edge
Parts:
- added 16MHz1: Crystal, Compluino_03:Crystal, F.Cu at (89.3, 122.3)
- added C1: 22pF, Capacitor_SMD:C_0805_2012Metric_Pad1.15x1.40mm_HandSolder, F.Cu at (133.4, 72.2)
- added C10: e1uF, Capacitor_SMD:CP_Elec_4x5.3, F.Cu at (197.1, 62.7)
- added C11: 100nF, Capacitor_SMD:C_0805_2012Metric_Pad1.15x1.40mm_HandSolder, F.Cu at (95.1, 126.1)
- added C12: 220nF, Capacitor_SMD:C_0805_2012Metric_Pad1.15x1.40mm_HandSolder, F.Cu at (144.2, 107.0)
- added C13: 100nF, Capacitor_SMD:C_0805_2012Metric_Pad1.15x1.40mm_HandSolder, F.Cu at (198.2, 81.2)
- added C14: 100nF, Capacitor_SMD:C_0805_2012Metric_Pad1.15x1.40mm_HandSolder, F.Cu at (170.8, 109.6)
- added C15: 100nF, Capacitor_SMD:C_0805_2012Metric_Pad1.15x1.40mm_HandSolder, F.Cu at (184.2, 93.4)
- added C16: 100nF, Capacitor_SMD:C_0805_2012Metric_Pad1.15x1.40mm_HandSolder, F.Cu at (157.4, 120.2)
- added C17: 100nF, Capacitor_SMD:C_0805_2012Metric_Pad1.15x1.40mm_HandSolder, F.Cu at (170.8, 107.6)
- added C18: 100nF, Capacitor_SMD:C_0805_2012Metric_Pad1.15x1.40mm_HandSolder, F.Cu at (175.7, 102.9)
- added C19: 100nF, Capacitor_SMD:C_0805_2012Metric_Pad1.15x1.40mm_HandSolder, F.Cu at (182.2, 96.3)
- added C2: 22pF, Capacitor_SMD:C_0805_2012Metric_Pad1.15x1.40mm_HandSolder, F.Cu at (105.8, 99.6)
- added C20: 100nF, Capacitor_SMD:C_0805_2012Metric_Pad1.15x1.40mm_HandSolder, F.Cu at (188.0, 91.5)
- added C21: 100nF, Capacitor_SMD:C_0805_2012Metric_Pad1.15x1.40mm_HandSolder, F.Cu at (153.1, 126.0)
- added C22: 100nF, Capacitor_SMD:C_0805_2012Metric_Pad1.15x1.40mm_HandSolder, F.Cu at (167.8, 111.6)
- added C23: 100nF, Capacitor_SMD:C_0805_2012Metric_Pad1.15x1.40mm_HandSolder, F.Cu at (177.8, 100.9)
- added C24: 100nF, Capacitor_SMD:C_0805_2012Metric_Pad1.15x1.40mm_HandSolder, F.Cu at (164.0, 113.6)
- added C25: 100nF, Capacitor_SMD:C_0805_2012Metric_Pad1.15x1.40mm_HandSolder, F.Cu at (193.2, 85.6)
- added C26: 100nF, Capacitor_SMD:C_0805_2012Metric_Pad1.15x1.40mm_HandSolder, F.Cu at (203.0, 76.0)
- added C27: 100nF, Capacitor_SMD:C_0805_2012Metric_Pad1.15x1.40mm_HandSolder, F.Cu at (157.4, 122.1)
- added C28: 100nF, Capacitor_SMD:C_0805_2012Metric_Pad1.15x1.40mm_HandSolder, F.Cu at (181.6, 98.2)
- added C29: e1uF, Capacitor_SMD:CP_Elec_4x5.3, F.Cu at (183.3, 79.1)
- added C3: e47uF, Capacitor_SMD:CP_Elec_6.3x5.3, F.Cu at (141.4, 113.1)
- added C30: e1uF, Capacitor_SMD:CP_Elec_4x5.3, F.Cu at (149.6, 113.3)
- added C31: e47uF, Capacitor_SMD:CP_Elec_6.3x5.3, F.Cu at (198.6, 56.7)
- added C32: 100nF, Capacitor_SMD:C_0805_2012Metric_Pad1.15x1.40mm_HandSolder, F.Cu at (91.3, 126.1)
- added C33: e47uF, Capacitor_SMD:CP_Elec_6.3x5.3, F.Cu at (175.1, 81.2)
- added C34: 100nF, Capacitor_SMD:C_0805_2012Metric_Pad1.15x1.40mm_HandSolder, F.Cu at (137.2, 72.2)
- added C35: e47uF, Capacitor_SMD:CP_Elec_6.3x5.3, F.Cu at (175.1, 74.0)
- added C36: 100nF, Capacitor_SMD:C_0805_2012Metric_Pad1.15x1.40mm_HandSolder, F.Cu at (87.6, 126.1)
- added C4: 100nF, Capacitor_SMD:C_0805_2012Metric_Pad1.15x1.40mm_HandSolder, F.Cu at (109.5, 99.6)
- added C5: e100nF, Capacitor_SMD:CP_Elec_4x5.3, F.Cu at (89.1, 116.5)
- added C6: e100nF, Capacitor_SMD:CP_Elec_4x5.3, F.Cu at (125.4, 94.6)
- added C7: e100nF, Capacitor_SMD:CP_Elec_4x5.3, F.Cu at (168.0, 91.0)
- added C8: e100nF, Capacitor_SMD:CP_Elec_4x5.3, F.Cu at (149.6, 108.4)
- added C9: e1uF, Capacitor_SMD:CP_Elec_4x5.3, F.Cu at (188.8, 71.7)
- added D2: LED, LED_SMD:LED_1210_3225Metric_Pad1.42x2.65mm_HandSolder, F.Cu at (199.9, 73.3)
- added D3: D, other:DO-214AA, F.Cu at (179.5, 93.3)
- added D4: D, other:DO-214AA, F.Cu at (173.0, 99.9)
- added D5: D, other:DO-214AA, F.Cu at (189.6, 82.7)
- added D6: D, other:DO-214AA, F.Cu at (144.3, 125.2)
- added D7: D, other:DO-214AA, F.Cu at (184.7, 86.6)
- added J12: Conn_01x04_OLED, Compluino_03:OLED, F.Cu at (107.2, 66.8)
- added J29: HOLE1, huellas:hole, F.Cu at (149.3, 124.3)
- added J30: HOLE2, huellas:hole, F.Cu at (160.1, 111.3)
- added J31: HOLE3, huellas:hole, F.Cu at (160.1, 115.3)
- added J32: HOLE4, huellas:hole, F.Cu at (166.9, 108.7)
- added J37: Conn_01x02_INPUT, proyectoAjeno:XT30PW-F2, F.Cu at (187.2, 67.3)
- added LED1: WS2812B, WS2812B:WS2812B_data-bridgeable, F.Cu at (167.5, 96.8)
- added LED10: WS2812B, WS2812B:WS2812B_data-bridgeable, F.Cu at (132.7, 123.0)
- added LED11: WS2812B, WS2812B:WS2812B_data-bridgeable, F.Cu at (167.5, 103.4)
- added LED12: WS2812B, WS2812B:WS2812B_data-bridgeable, F.Cu at (194.8, 75.0)
- added LED13: WS2812B, WS2812B:WS2812B_data-bridgeable, F.Cu at (162.3, 106.0)
- added LED14: WS2812B, WS2812B:WS2812B_data-bridgeable, F.Cu at (149.2, 119.0)
- added LED15: WS2812B, WS2812B:WS2812B_data-bridgeable, F.Cu at (189.3, 77.4)
- added LED16: WS2812B, WS2812B:WS2812B_data-bridgeable, F.Cu at (203.1, 63.5)
- added LED2: WS2812B, WS2812B:WS2812B_data-bridgeable, F.Cu at (179.1, 88.1)
- added LED3: WS2812B, WS2812B:WS2812B_data-bridgeable, F.Cu at (144.0, 120.0)
- added LED4: WS2812B, WS2812B:WS2812B_data-bridgeable, F.Cu at (173.9, 88.1)
- added LED5: WS2812B, WS2812B:WS2812B_data-bridgeable, F.Cu at (155.5, 109.3)
- added LED6: WS2812B, WS2812B:WS2812B_data-bridgeable, F.Cu at (196.4, 68.4)
- added LED7: WS2812B, WS2812B:WS2812B_data-bridgeable, F.Cu at (162.3, 99.4)
- added LED8: WS2812B, WS2812B:WS2812B_data-bridgeable, F.Cu at (173.9, 94.7)
- added LED9: WS2812B, WS2812B:WS2812B_data-bridgeable, F.Cu at (155.5, 115.9)
- added Q1: IRF540N, other:D2PAK, F.Cu at (164.0, 76.3)
- added Q2: IRF540N, other:D2PAK, F.Cu at (136.0, 97.2)
- added Q3: IRF540N, other:D2PAK, F.Cu at (174.2, 58.2)
- added R10: 10K, Resistor_SMD:R_0805_2012Metric_Pad1.15x1.40mm_HandSolder, F.Cu at (177.8, 98.9)
- added R11: 1K, Resistor_SMD:R_0805_2012Metric_Pad1.15x1.40mm_HandSolder, F.Cu at (172.0, 104.8)
- added R12: 10K, Resistor_SMD:R_0805_2012Metric_Pad1.15x1.40mm_HandSolder, F.Cu at (187.4, 89.5)
- added R13: 1K, Resistor_SMD:R_0805_2012Metric_Pad1.15x1.40mm_HandSolder, F.Cu at (197.5, 79.3)
- added R14: 10K, Resistor_SMD:R_0805_2012Metric_Pad1.15x1.40mm_HandSolder, F.Cu at (164.0, 111.6)
- added R15: 1K, Resistor_SMD:R_0805_2012Metric_Pad1.15x1.40mm_HandSolder, F.Cu at (194.4, 83.2)
- added R16: 249, Resistor_SMD:R_0805_2012Metric_Pad1.15x1.40mm_HandSolder, F.Cu at (189.4, 87.6)
- added R17: 11,3K, Resistor_SMD:R_0805_2012Metric_Pad1.15x1.40mm_HandSolder, F.Cu at (153.1, 124.1)
- added R18: 11,3K, Resistor_SMD:R_0805_2012Metric_Pad1.15x1.40mm_HandSolder, F.Cu at (172.0, 102.9)
- added R19: 11,3K, Resistor_SMD:R_0805_2012Metric_Pad1.15x1.40mm_HandSolder, F.Cu at (127.1, 117.7)
- added R2: 10K, Resistor_SMD:R_0805_2012Metric_Pad1.15x1.40mm_HandSolder, F.Cu at (153.7, 120.2)
- added R20: 11,3K, Resistor_SMD:R_0805_2012Metric_Pad1.15x1.40mm_HandSolder, F.Cu at (175.7, 104.8)
- added R21: 1K, Resistor_SMD:R_0805_2012Metric_Pad1.15x1.40mm_HandSolder, F.Cu at (191.1, 89.5)
- added R22: 1K, Resistor_SMD:R_0805_2012Metric_Pad1.15x1.40mm_HandSolder, F.Cu at (201.3, 77.9)
- added R23: 1K, Resistor_SMD:R_0805_2012Metric_Pad1.15x1.40mm_HandSolder, F.Cu at (189.4, 85.6)
- added R24: 1K, Resistor_SMD:R_0805_2012Metric_Pad1.15x1.40mm_HandSolder, F.Cu at (181.8, 82.5)
- added R25: 10K, Resistor_SMD:R_0805_2012Metric_Pad1.15x1.40mm_HandSolder, F.Cu at (193.8, 79.3)
- added R3: 10K, Resistor_SMD:R_0805_2012Metric_Pad1.15x1.40mm_HandSolder, F.Cu at (164.0, 115.5)
- added R4: 10K, Resistor_SMD:R_0805_2012Metric_Pad1.15x1.40mm_HandSolder, F.Cu at (178.4, 96.3)
- added R5: 10K, Resistor_SMD:R_0805_2012Metric_Pad1.15x1.40mm_HandSolder, F.Cu at (184.2, 91.5)
- added R6: 2K, Resistor_SMD:R_0805_2012Metric_Pad1.15x1.40mm_HandSolder, F.Cu at (153.7, 122.1)
- added R7: 1K, Resistor_SMD:R_0805_2012Metric_Pad1.15x1.40mm_HandSolder, F.Cu at (199.3, 76.0)
- added R8: 10k, Resistor_SMD:R_0805_2012Metric_Pad1.15x1.40mm_HandSolder, F.Cu at (137.2, 125.1)
- added R9: 10K, Resistor_SMD:R_0805_2012Metric_Pad1.15x1.40mm_HandSolder, F.Cu at (194.4, 81.2)
- added RV1: R_POT, Compluino_03:Potenciometro, F.Cu at (148.9, 76.9)
- added SW1: RESET, huellas:PULSADOR, F.Cu at (158.8, 62.2)
- added SW10: SW_DIP_x08, huellas:SWITCH, F.Cu at (79.6, 115.0)
- added SW5: UP, huellas:PULSADOR, F.Cu at (131.1, 83.1)
- added SW6: RIGHT, huellas:PULSADOR, F.Cu at (140.6, 62.2)
- added SW7: LEFT, huellas:PULSADOR, F.Cu at (102.4, 110.4)
- added SW8: OK, huellas:PULSADOR, F.Cu at (113.0, 89.5)
- added SW9: DOWN, huellas:PULSADOR, F.Cu at (120.6, 107.7)
- added U1: ATmega2560-16AU, Package_QFP:TQFP-100_14x14mm_P0.5mm, F.Cu at (151.0, 97.3)
- added U10: LM2907, LM2907:SOIC8, F.Cu at (183.0, 73.0)
- added U11: LM2907, LM2907:SOIC8, F.Cu at (162.2, 92.3)
- added U12: L7805, Compluino_03:7805, F.Cu at (123.7, 72.8)
- added U13: L7805, Compluino_03:7805, F.Cu at (96.1, 100.2)
- added U2: 74LS247, other:SO16, F.Cu at (103.0, 123.4)
- added U3: CC56-12SYKWA, Display_7Segment:CA56-12SYKWA, F.Cu at (76.0, 72.2)
- added U4: HEF4040BT, HEF4040BT:SOIC127P600X175-16N, F.Cu at (115.0, 121.8)
- added U5: HEF4040BT, HEF4040BT:SOIC127P600X175-16N, F.Cu at (89.1, 109.0)
- added U6: HEF4040BT, HEF4040BT:SOIC127P600X175-16N, F.Cu at (133.1, 114.6)
- added U7: HEF4040BT, HEF4040BT:SOIC127P600X175-16N, F.Cu at (121.8, 121.8)
- added U8: LM2907, LM2907:SOIC8, F.Cu at (139.0, 120.4)
- added U9: LM2907, LM2907:SOIC8, F.Cu at (127.7, 123.4)
- D1: footprint LED_SMD:LED_1206_3216Metric_Pad1.42x1.75mm_HandSolder -> LED_SMD:LED_1210_3225Metric_Pad1.42x2.65mm_HandSolder
- R1: value R -> 249; footprint Resistor_SMD:R_1206_3216Metric_Pad1.42x1.75mm_HandSolder -> Resistor_SMD:R_0805_2012Metric_Pad1.15x1.40mm_HandSolder
- moved D1 61.4 mm to (201.5, 68.5)
- moved R1 47.7 mm to (183.6, 89.5), turned to 0 degrees
Connections:
- D1 pad 1: +5V -> Net-(D1-Pad1)
- D1 pad 2: Net-(D1-Pad2) -> +5V
- R1 pad 1: Net-(D1-Pad2) -> Earth
- R1 pad 2: Earth -> Net-(D1-Pad1)
Routing:
- net Net-(D1-Pad2): track 12.6 -> 0.00 mm

Commit message: placa ATtiny1634
Connections:
- C12 pad 2: RESET_Bluetooth -> RESET_FTDI
- R25 pad 1: +5V -> +5VP
