File: ELECTRONICA/ATtiny_2.0/ATtiny_2.0.sch (KiCad schematic (older format))
At the start: 23 parts, among them J1 Puerto_Temperatura_1, J12 XT30, J2 ICSP, J3 I2C, J4 UART0, J5 Puerto Motores, J6 Puerto_Temperatura_1, SW1 SW_Push, U1 ATtiny1634-SU, U2 L7805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

Commit message: Desarrollo de la Tiny 2.0
Parts:
- removed R5, R6: R10K, Resistor_SMD:R_0805_2012Metric_Pad1.15x1.40mm_HandSolder, symbol Device:R
- added J13: GND, Connector_PinHeader_2.54mm:PinHeader_1x04_P2.54mm_Vertical, symbol Connector_Generic:Conn_01x04
- added J14: VCC, Connector_PinHeader_2.54mm:PinHeader_1x04_P2.54mm_Vertical, symbol Connector_Generic:Conn_01x04
- added J4: I2C1, Connector_PinHeader_2.54mm:PinHeader_1x04_P2.54mm_Vertical, symbol Connector_Generic:Conn_01x04
- added J7: Puerto_Encoders, Connector_PinHeader_2.54mm:PinHeader_1x02_P2.54mm_Vertical, symbol Connector_Generic:Conn_01x02
- added R10, R12, R7, R8, R9: R10K, Resistor_SMD:R_0805_2012Metric_Pad1.15x1.40mm_HandSolder, symbol Device:R
- added R11: R1K, Resistor_SMD:R_0805_2012Metric_Pad1.15x1.40mm_HandSolder, symbol Device:R
- added R13: R100K, Resistor_SMD:R_0805_2012Metric_Pad1.15x1.40mm_HandSolder, symbol Device:R
- added SW2: SW_DIP_x04, Button_Switch_SMD:SW_DIP_SPSTx04_Slide_6.7x11.72mm_W6.73mm_P2.54mm_LowProfile_JPin, symbol Switch:SW_DIP_x04
- J2: renamed from J6; value Puerto_Temperatura_1 -> Puerto_Temperatura_2
- J3: value I2C -> I2C0
- renumbered J4 to J6, J2 to J8
Connections:
- net PB3 is gone; now on net TEMP1: U1.18 (PB3)
- net PC0 is gone; now on net TEMP2: U1.17 (PC0)
- net +5V: now also J5.3 (Pin_3), J14.1 (Pin_1), J14.2 (Pin_2), J14.3 (Pin_3), J14.4 (Pin_4), J4.1 (Pin_1), R11.1, R12.1, R7.2, R8.1
- net CS: now also U1.7 (PA2); no longer U1.6 (PA3)
- net Earth: now also J13.1 (Pin_1), J13.2 (Pin_2), J13.3 (Pin_3), J13.4 (Pin_4), J4.4 (Pin_4), R13.2
- net MOSI-SDA-RX1: now also J4.2 (Pin_2), R8.2
- net SCK-SCL: now also J4.3 (Pin_3), R7.1
- net TEMP1: no longer U1.9 (AREF/PA0)
- net TEMP2: no longer U1.8 (PA1)
- removed net EN: J5.3 (Pin_3), U1.7 (PA2)
- net INA renamed D1
- net D1: now also J5.6 (Pin_6); no longer J5.5 (Pin_5)
- net INB: no longer names the net of U1.3 (PA6)
- net INB: now also R2.1; no longer J5.6 (Pin_6)
- net PC2 renamed SWITCH
- net SWITCH: now also R13.1, SW2.1, SW2.2; no longer R2.1
- new net: J7.1 (Pin_1), R10.2
- new net: J7.2 (Pin_2), R9.1
- new net: R11.2, SW2.8
- new net: R12.2, SW2.7
- new net D2: J5.5 (Pin_5), U1.6 (PA3)
- new net INT1: R10.1, U1.8 (PA1)
- new net INT2: R9.2, U1.9 (AREF/PA0)
Other:
- moved on the sheet: D2, J3, J6, R2
