File: ELECTRONICA/ATtiny_3.0/ATtiny_3.0.kicad_pcb (KiCad board)
At the start: 2 copper layers, 38 parts, among them J1 ICSP, J12 XT30, J2 I2C_IN, J3 JUMPER1, J4 JUMPER2, J5 Puerto Motores, J6 I2C_OUT, J7 Puerto_Encoders, SW1 SW_Push, U1 ATtiny1634-SU, U2 L7805, Y1 Crystal 16MHz

Commit message: odom
Parts:
- removed J2: I2C_IN, Connector_PinHeader_2.54mm:PinHeader_1x03_P2.54mm_Vertical
- removed J6: I2C_OUT, Connector_PinHeader_2.54mm:PinHeader_1x03_P2.54mm_Vertical
- removed J7: Puerto_Encoders, Connector_PinHeader_2.54mm:PinHeader_1x02_P2.54mm_Vertical
- added  : I2C_IN, Connector_Molex:Molex_KK-254_AE-6410-04A_1x04_P2.54mm_Vertical, F.Cu at (128.7, 60.2)
- added  : I2C_OUT, Connector_Molex:Molex_KK-254_AE-6410-04A_1x04_P2.54mm_Vertical, F.Cu at (128.7, 67.2)
- added  : Puerto_Encoders, Connector_Molex:Molex_KK-254_AE-6410-04A_1x04_P2.54mm_Vertical, F.Cu at (131.1, 81.6)
- added G***: LOGO, huellas:zebra_n, B.Cu at (115.8, 69.3)
-  : renamed from J12
-  : renamed from J3
-  : renamed from J4
-  : renamed from J5
-  : renamed from SW1
-  : renamed from H1
-  : renamed from H2
-  : renamed from H3
-  : renamed from H4
-  : renamed from H5
-  : renamed from H6
-  : renamed from H7
-  : renamed from H8
- moved R1 179.6 mm to (134.6, 44.5)
- moved R7 170.2 mm to (124.5, 64.8), turned to 180 degrees
- moved R4 154.7 mm to (124.5, 89.6)
- moved R5 144.9 mm to (124.5, 73.7)
- moved ATtiny1634 143.0 mm to (111.8, 81.3)
- moved   142.5 mm to (136.0, 34.8)
- moved ICSP 138.8 mm to (130.8, 49.5)
- moved R2 138.8 mm to (100.3, 64.8), turned to 180 degrees
- moved R8 138.5 mm to (124.5, 62.2)
- moved LED1 137.7 mm to (98.2, 41.7), turned to 270 degrees
- moved R3 134.6 mm to (100.3, 67.3), turned to 180 degrees
- moved R10 132.0 mm to (124.5, 82.4)
- moved R9 131.8 mm to (124.5, 84.9)
- moved LED2 130.7 mm to (95.0, 41.7), turned to 270 degrees
- moved C3 127.1 mm to (109.2, 60.0)
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- renumbered U1 to ATtiny1634, Y1 to CLK, J1 to ICSP, U2 to L7805, D1 to LED1, D2 to LED2, D0 to POWER
Connections:
- R5 pad 1: Earth -> +5V
- R6 pad 1: Earth -> +5V
Routing:
- net Earth: track 0.00 -> 217.9 mm, vias 0 -> 1
- net +5V: track 0.00 -> 168.5 mm, vias 0 -> 3
- net SCK-SCL: track 0.00 -> 60.3 mm, vias 0 -> 2
- net RESET: track 0.00 -> 58.9 mm, vias 0 -> 3
- net INT1: track 0.00 -> 55.2 mm, vias 0 -> 2
- net MOSI-SDA: track 0.00 -> 51.7 mm, vias 0 -> 1
- net DIRECTION1: track 0.00 -> 46.7 mm, vias 0 -> 1
- net DIRECTION2: track 0.00 -> 40.9 mm, vias 0 -> 1
- net MISO: track 0.00 -> 36.1 mm
- net Net-(C3-Pad2): track 0.00 -> 35.0 mm
- net HANDSHAKE: track 0.00 -> 35.0 mm, vias 0 -> 1
- net Net-(C4-Pad2): track 0.00 -> 31.9 mm
- net Net-(D2-Pad2): track 0.00 -> 28.1 mm
- net Net-(R3-Pad1): track 0.00 -> 27.7 mm, vias 0 -> 2
- net Net-(R2-Pad1): track 0.00 -> 27.3 mm
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Other:
- board outline added: 47 x 75.6 mm
- net class Power added: clearance 0.2, trace_width 0.7, via_dia 1.3, via_drill 0.9
- board text added: "+5V"
- board text added: "CS"
- board text added: "CuagaForce Board v3.0"
- board text added: "DIR1"
- board text added: "DIR2"
- board text added: "EN"
- board text added: "G"
- board text added: "GND"
- board text added: "H"
- board text added: "INA"
- board text added: "INB"
- board text added: "INT1"
- board text added: "INT2"
- board text added: "MISO"
- board text added: "MOSI"
- board text added: "PWM"
- board text added: "RESET"
- board text added: "RST"
- board text added: "SCK"
- board text added: "SCL"
- board text added: "SDA"
- board text added: "VCC"
